File: design_files/AST1042.brd (EAGLE design)
At the start: 12 x 14 mm, 11 parts, among them J1 SM05B, U1 RGC04072040

Commit message: update naming
Parts:
- C2: value 10uF -> 1uF
- J1: device tinycircuits:JST_SH_5X1 -> tinycircuits:JST_SH_5X1_EDGE
- R2: value 0.0 -> 1.00K
Other:
- outline, holes or cut-outs redrawn
- board text added: "Wireling 0.42 OLED"
- board text removed: "0.42" OLED"
Changed lines of the file:
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@@
 <setting verticaltext="up"/>
 </settings>
-<grid distance="0.1" unitdist="mm" unit="mm" style="lines" multiple="1" display="yes" altdistance="0.1" altunitdist="mm" altunit="mm"/>
+<grid distance="0.5" unitdist="mm" unit="mm" style="lines" multiple="1" display="yes" altdistance="0.1" altunitdist="mm" altunit="mm"/>
 <layers>
 <layer number="1" name="Top" color="4" fill="1" visible="yes" active="yes"/>
@@
 <layer number="158" name="bResistor" color="7" fill="1" visible="no" active="yes"/>
 <layer number="159" name="henwayCAP" color="13" fill="1" visible="yes" active="yes"/>
+<layer number="160" name="IDFDebug" color="7" fill="1" visible="yes" active="yes"/>
 <layer number="191" name="mNets" color="7" fill="1" visible="no" active="no"/>
 <layer number="192" name="mBusses" color="7" fill="1" visible="no" active="no"/>
@@
 <wire x1="0" y1="45.8" x2="0" y2="0" width="0.127" layer="48"/>
 <dimension x1="17.5" y1="29" x2="29.5" y2="29" x3="23.5" y3="34.15465" layer="48"/>
-<text x="51.111025" y="4.365003125" size="0.889" layer="48">0.42" OLED</text>
+<text x="51.111025" y="4.365003125" size="0.889" layer="48">Wireling 0.42 OLED</text>
 <text x="47.986825" y="1.7714" size="0.889" layer="48">AS-PCB-AST1042</text>
 <text x="70.3810375" y="1.6952" size="0.889" layer="48">1</text>
@@
 <wire x1="17.5" y1="29" x2="17.5" y2="15" width="0.0254" layer="20"/>
 <dimension x1="17.5" y1="29" x2="17.5" y2="15" x3="10.7" y3="22" layer="48"/>
-<wire x1="29.5" y1="29" x2="26.5" y2="29" width="0.0254" layer="20"/>
-<wire x1="26.5" y1="29" x2="26.5" y2="26" width="0.0254" layer="20"/>
-<wire x1="26.5" y1="26" x2="20.5" y2="26" width="0.0254" layer="20"/>
-<wire x1="20.5" y1="26" x2="20.5" y2="29" width="0.0254" layer="20"/>
-<wire x1="20.5" y1="29" x2="17.5" y2="29" width="0.0254" layer="20"/>
+<wire x1="29.5" y1="29" x2="26" y2="29" width="0.0254" layer="20"/>
+<wire x1="26.5" y1="28.5" x2="26.5" y2="26.5" width="0.0254" layer="20"/>
+<wire x1="26" y1="26" x2="21" y2="26" width="0.0254" layer="20"/>
+<wire x1="20.5" y1="26.5" x2="20.5" y2="28.5" width="0.0254" layer="20"/>
+<wire x1="20.5" y1="28.5" x2="21" y2="29" width="0.0254" layer="20" curve="-90"/>
+<wire x1="21" y1="29" x2="17.5" y2="29" width="0.0254" layer="20"/>
 <text x="43.0812" y="14.456396875" size="0.4572" layer="48" ratio="10">Released under the Creative Commons Attribution Share-Alike 3.0 License</text>
 <text x="43.0812" y="13.795996875" size="0.4572" layer="48" ratio="10">http://creativecommons.org/licenses/by-sa/3.0</text>
@@
 <hole x="28" y="27.5" drill="1.5"/>
 <text x="18.7" y="23.7" size="0.762" layer="21" rot="SR90">1042</text>
+<wire x1="21" y1="26" x2="20.5" y2="26.5" width="0.0254" layer="20" curve="-90"/>
+<wire x1="26.5" y1="26.5" x2="26" y2="26" width="0.0254" layer="20" curve="-90"/>
+<wire x1="26" y1="29" x2="26.5" y2="28.5" width="0.0254" layer="20" curve="-90"/>
 </plain>
 <attributes>
@@
 <attribute name="VALUE" value="0.1uF" x="22.15" y="21.95" size="1.778" layer="27" rot="R180" display="off"/>
 </element>
-<element name="C2" library="tinycircuits" package="C0603" value="10uF" x="22.3" y="23.1" rot="R180">
-<attribute name="PARTNO" value="AS-ITM-00002" x="22.3" y="23.1" size="1.778" layer="27" rot="R180" display="off"/>
-<attribute name="VALUE" value="10uF" x="22.3" y="23.1" size="1.778" layer="27" rot="R180" display="off"/>
+<element name="C2" library="tinycircuits" package="C0603" value="1uF" x="22.3" y="23.1" rot="R180">
+<attribute name="PARTNO" value="AS-ITM-00410" x="22.3" y="23.1" size="1.778" layer="27" rot="R180" display="off"/>
+<attribute name="VALUE" value="1uF" x="22.3" y="23.1" size="1.778" layer="27" rot="R180" display="off"/>
 </element>
-<element name="J1" library="tinycircuits" package="JST_SH_5X1" value="SM05B" x="23.5" y="17.225">
+<element name="J1" library="tinycircuits" package="JST_SH_5X1_EDGE" value="SM05B" x="23.5" y="17.225">
 <attribute name="PARTNO" value="AS-ITM-00340" x="23.5" y="17.225" size="1.778" layer="27" display="off"/>
 <attribute name="VALUE" value="SM05B" x="23.5" y="17.225" size="1.778" layer="27" display="off"/>
@@
 <attribute name="VALUE" value="1uF" x="19.4" y="20.9" size="1.778" layer="27" display="off"/>
 </element>
-<element name="R2" library="tinycircuits" package="0402" value="0.0" x="25.4" y="23.1" rot="R90">
-<attribute name="PARTNO" value="AS-ITM-00076" x="25.4" y="23.1" size="1.778" layer="27" rot="R90" display="off"/>
-<attribute name="VALUE" value="0.0" x="25.4" y="23.1" size="1.778" layer="27" rot="R90" display="off"/>
+<element name="R2" library="tinycircuits" package="0402" value="1.00K" x="25.4" y="23.1" rot="R90">
+<attribute name="PARTNO" value="AS-ITM-00003" x="25.4" y="23.1" size="1.778" layer="27" rot="R90" display="off"/>
+<attribute name="VALUE" value="1.00K" x="25.4" y="23.1" size="1.778" layer="27" rot="R90" display="off"/>
 </element>
 <element name="C5" library="tinycircuits" package="C0805" value="10uF" x="28.2" y="18.6" rot="R270">
