File: design_files/AST1042.sch (EAGLE design)
At the start: 10 parts, among them J1 SM05B, U1 RGC04072040

Commit message: update naming
Parts:
- C2: value 10uF -> 1uF; device tinycircuits:AS-ITM-00002 -> tinycircuits:AS-ITM-00410; PARTNO (none) -> AS-ITM-00410; VALUE (none) -> 1uF
- J1: device tinycircuits:AS-ITM-00340 -> tinycircuits:AS-ITM-00340EDGE
- R2: value 0.0 -> 1.00K; device tinycircuits:AS-ITM-00076 -> tinycircuits:AS-ITM-00003; PARTNO (none) -> AS-ITM-00003; VALUE (none) -> 1.00K
Other:
- note added: "0.42" OLED Display"
- note added: "Wireling 0.42 OLED"
- note removed: "0.42" OLED"
- note removed: "0.49" OLED Display"
